File: p1/Kit-Trig-Sampler.kicad_sch (KiCad schematic)
At the start: 126 parts, among them CON1 microSDCon_Vert_TH_PJS008U-30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, IC1 TL082, IC2 TL082, IC3 TL082, J1 3.5mm_Mono_Switched, J2 3.5mm_Mono_Switched, J3 3.5mm_Mono_Switched, J4 3.5mm_Mono_Switched, J5 3.5mm_Mono_Switched, J6 3.5mm_Mono_Switched, J7 3.5mm_Mono_Switched, J8 3.5mm_Mono_Switched, P1 Pins_02x05_TH, U11 white, U12 blue, U13 PCA9685, U14 SW_PUSH_SMALL, U18 PCA9685, U4 CONN_02X10, U5 16mm_CtrDet_10k, U6 16mm_NoDet_10k, U7 16mm_NoDet_10k, U8 16mm_NoDet_10k, U9 16mm_NoDet_10k

Commit message: STS kit
schematic drawin
Parts:
- removed C11, C12, C3: 10nF_0805_50V, 4ms_Capacitor:C_0805, symbol 4ms_Capacitor:10nF_0805_50V
- removed C2, C6, C7: 1nF_0603_50V, 4ms_Capacitor:C_0603, symbol 4ms_Capacitor:1nF_0603_50V
- removed C22: 1uF_0805_25V, 4ms_Capacitor:C_0805, symbol 4ms_Capacitor:1uF_0805_25V
- removed C30, C32, C4, C8, C9: 0.1uF_0805_50V, 4ms_Capacitor:C_0805, symbol 4ms_Capacitor:0.1uF_0805_50V
- removed D1, D2, D3, D4, D6, D7: BAT54S, 4ms_Package_SOT:SOT23-3_PO132, symbol 4ms_Diode:BAT54S
- removed unit 2 of IC1
- removed unit 1 of IC1
- removed unit 1 of IC3
- removed J8: 3.5mm_Mono_Switched, 4ms_Jack:EighthInch_PJ398SM, symbol 4ms_Jack:3.5mm_Mono_Switched
- removed R23, R27: 100k_0805, 4ms_Resistor:R_0805, symbol 4ms_Resistor_0805:100k_0805
- removed R26, R28: 1M_0805, 4ms_Resistor:R_0805, symbol 4ms_Resistor:1M_0805
- removed R30, R40, R42, R5, R50, R52: 1k_0805, 4ms_Resistor:R_0805, symbol 4ms_Resistor:1k_0805
- removed R37, R45: 4.7k_0805, 4ms_Resistor:R_0805, symbol 4ms_Resistor_0805:4.7k_0805
- removed R41, R51: 2.7k_0805, 4ms_Resistor:R_0805, symbol 4ms_Resistor_0805:2.7k_0805
- removed S3, S5: Button_SPST_RGB_5.4mmCap, 4ms_Switch:Button_RgbLED_SPST_PB615303HL-7mm, symbol 4ms_Switch:Button_SPST_RGB_5.4mmCap
- removed U12: blue, 4ms-footprints:LED-3MM-SQUARE-ANODE, symbol TrigSampler-rescue:LED-RESCUE-TrigSampler
- removed U14: SW_PUSH_SMALL, 4ms-footprints:SPST-SUB, symbol TrigSampler-rescue:SW_PUSH_SMALL
- removed U18: PCA9685, 4ms-footprints:TSSOP-28_4.4x9.7mm_Pitch0.65mm, symbol TrigSampler-rescue:PCA9685
- removed U8: 16mm_NoDet_10k, 4ms_Potentiometer:Pot_16mm_NoDet_RV16AF-4A, symbol 4ms_Potentiometer:16mm_NoDet_10k
- added C?: 470pF, 4ms-footprints:C0603, symbol TrigSampler-rescue:C_Small
- added C?: 2.7nF, 4ms-footprints:C0603, symbol TrigSampler-rescue:C_Small
- added C?: 4.7nF, 4ms-footprints:C0603, symbol TrigSampler-rescue:C_Small
- added IC?: NJM2068, 4ms-footprints:TSSOP-8_4.4x3mm_Pitch0.65mm, symbol TrigSampler-rescue:NJM2068-dualpwr
- added J?: OUT-1, 4ms-footprints:PJ301M-12, symbol TrigSampler-rescue:JACK-MONO
- added R?: 715, 4ms-footprints:R0603, symbol TrigSampler-rescue:R
- added R?: 1.5k, 4ms-footprints:R0603, symbol TrigSampler-rescue:R
- added R?: 7.15k, 4ms-footprints:R0603, symbol TrigSampler-rescue:R
- added R?: 1.2k, 4ms-footprints:R0603, symbol TrigSampler-rescue:R
- added R?: 7.87k, 4ms-footprints:R0603, symbol TrigSampler-rescue:R
- added R?: 1k, 4ms-footprints:R0603, symbol TrigSampler-rescue:R
- added R?: 2.7k, 4ms-footprints:R0603, symbol TrigSampler-rescue:R
- C1, C25, C26, C28, C29, C31: footprint 4ms_Capacitor:C_0805 -> 4ms_Capacitor:C_Disc_P2.54mm; symbol 4ms_Capacitor:0.1uF_0805_50V -> 4ms_Capacitor:0.1uF_Disc_TH; Display 0.1uF/50V -> 0.1uF
- C13, C14, C15, C16, C17, C18: footprint 4ms_Capacitor:C_0805 -> 4ms_Capacitor:C_Disc_P2.54mm; symbol 4ms_Capacitor:0.1uF_0805_50V -> 4ms_Capacitor:0.1uF_Disc_TH
- C5: footprint 4ms_Capacitor:C_0603 -> 4ms_Capacitor:C_Disc_P5.08mm
- IC1, IC2, IC3: footprint 4ms_Package_SSOP:TSSOP-8_4.4x3mm_Pitch0.65mm -> 4ms_Package_DIP:DIP-8pin_TH; symbol 4ms_IC:TL082 -> 4ms_IC:TL082_TH; Specifications TL082 Dual Opamp TSSOP-8 -> TL082 Dual Opamp DIP-8pin
- R1: value 600 -> 620; footprint 4ms-footprints:R0603 -> 4ms_Resistor:R_Axial_DIN0207_L6.3mm_D2.5mm_P7.62mm_Horizontal; symbol TrigSampler-rescue:R -> 4ms_Resistor_TH:620Ω_TH0.125; Display (none) -> 620Ω; Manufacturer (none) -> Xicon; Part Number (none) -> 299-620-RC; Specifications (none) -> 620Ω, 5%, 1/8W, TH0.125
- R17, R20, R21, R22, R25, R7, R8: footprint 4ms_Resistor:R_0805 -> 4ms_Resistor:R_Axial_DIN0207_L6.3mm_D2.5mm_P7.62mm_Horizontal; symbol 4ms_Resistor_0805:100k_0805 -> 4ms_Resistor_TH:100k_TH0.125; Manufacturer Yageo -> Xicon; Part Number RC0805FR-07100KL -> 299-100k-RC; Specifications 100k, 1%, 1/8W, 0805 -> 100k, 5%, 1/8W, TH0.125
- R18, R19, R3: footprint 4ms_Resistor:R_0805 -> 4ms_Resistor:R_Axial_DIN0207_L6.3mm_D2.5mm_P7.62mm_Horizontal; symbol 4ms_Resistor_0805:49.9k_0805 -> 4ms_Resistor_TH:47k_TH0.125; Display 49.9k -> 47k; Manufacturer Yageo -> Xicon; Part Number RC0805FR-0749K9L -> 299-47k-RC; Specifications 49.9k, 1%, 1/8W, 0805 -> 47k, 5%, 1/8W, TH0.125
- R2, R29, R32, R34, R36, R39, R4, R9: footprint 4ms_Resistor:R_0805 -> 4ms_Resistor:R_Axial_DIN0207_L6.3mm_D2.5mm_P7.62mm_Horizontal; symbol 4ms_Resistor:1k_0805 -> 4ms_Resistor_TH:1k_TH0.125; Manufacturer Yageo -> Xicon; Part Number RT0805FRE071KL -> 299-1k-RC; Specifications 1k, 1/8W, 1% -> 1k, 5%, 1/8W, TH0.125
Connections:
- net +3.3VADC: no longer R2.2
- net A0: now also R3.2, R7.2
- net A1: now also R18.2, R20.2
- net A2: now also C5.1, IC2.7, R15.1
- net A3: now also R19.2, R21.2
- net D0: now also J7.1 (SIG)
- net GND: now also C1.1, R1.1, R20.1, R21.1, R7.1, J?.2 (SHEILD)
- net GNDADC: no longer C1.1, R1.1, R20.1, R21.1, R7.1
- net VREF+: now also R2.2
- net BANKREC_B_LED: no longer names the net of U13.8 (LED2)
- net BANKREC_G_LED: no longer names the net of U13.7 (LED1)
- net BANKREC_R_LED: no longer names the net of U13.6 (LED0)
- net REC_B_LED: no longer names the net of U13.11 (LED5)
- net REC_G_LED: no longer names the net of U13.10 (LED4)
- net REC_R_LED: no longer names the net of U13.9 (LED3)
- new net: R?.1, R?.1, R?.2
- new net: C?.1, IC?.3 (+), R?.2
- new net: C?.1, IC?.2 (-), R?.1
- new net: C?.2, IC?.1, R?.1, R?.2
- new net: C?.2, R?.1, R?.1, R?.2
- new net: J?.1 (SIG), R?.2
- new net AOUTA1_M: R?.2
- new net AOUTA1_P: R?.1
- new net GNDA: C?.1, C?.2, R?.2
- no-connect marks 18 -> 20
Other:
- note added: "Analog Inputs"
- note added: "Digital Ins/Outs"
- note removed: "600R IS NOT STANDARD closest is 665R that ok?"
- note removed: "BankRec_But"
- note removed: "Edit_But"
- note removed: "RecSamp_Pot"
- note removed: "i consolidated the LEDx side of these two PCA chips but on the other side they are not exactly the same... tho close see pins 25 and A0 which config to use? can I consolidate these in the first place? Do these even belong here or is this a brainboard thing? Was not sure what to do here..."
- moved on the sheet: C1, C10, C13, C14, C15, C16, C17, C18, C26, C5, D5, IC1C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

Commit message: forgotten push
Parts:
- removed C10: 10nF_0805_50V, 4ms_Capacitor:C_0805, symbol 4ms_Capacitor:10nF_0805_50V
- removed C17, C18, C25, C28: 0.1uF_0805_50V, 4ms_Capacitor:C_Disc_P2.54mm, symbol 4ms_Capacitor:0.1uF_Disc_TH
- removed C24, C27: 47uF_5x5.3_16V, 4ms_Capacitor:CP_Elec_5x5.3, symbol 4ms_Capacitor:47uF_5x5.3_16V
- removed C?: 470pF, 4ms-footprints:C0603, symbol TrigSampler-rescue:C_Small
- removed C?: 2.7nF, 4ms-footprints:C0603, symbol TrigSampler-rescue:C_Small
- removed C?: 4.7nF, 4ms-footprints:C0603, symbol TrigSampler-rescue:C_Small
- removed D5: BAT54S, 4ms_Package_SOT:SOT23-3_PO132, symbol 4ms_Diode:BAT54S
- removed D8, D9: B140-E3, 4ms_Diode:D_SMA, symbol 4ms_Diode:B140-E3
- removed IC3: TL082, 4ms_Package_DIP:DIP-8pin_TH, symbol 4ms_IC:TL082_TH
- removed IC?: NJM2068, 4ms-footprints:TSSOP-8_4.4x3mm_Pitch0.65mm, symbol TrigSampler-rescue:NJM2068-dualpwr
- removed J3: 3.5mm_Mono_Switched, 4ms_Jack:EighthInch_PJ398SM, symbol 4ms_Jack:3.5mm_Mono_Switched
- removed J?: OUT-1, 4ms-footprints:PJ301M-12, symbol TrigSampler-rescue:JACK-MONO
- removed JA1: Header A, Connector_PinSocket_2.54mm:PinSocket_2x05_P2.54mm_Vertical_SMD, symbol 4ms_Connector:Pins_02x05_SMT
- removed JB1: Header B, Connector_PinSocket_2.54mm:PinSocket_2x05_P2.54mm_Vertical_SMD, symbol 4ms_Connector:Pins_02x05_SMT
- removed JC1: Header C, Connector_PinSocket_2.54mm:PinSocket_2x05_P2.54mm_Vertical_SMD, symbol 4ms_Connector:Pins_02x05_SMT
- removed JD1: Header D, Connector_PinSocket_2.54mm:PinSocket_2x05_P2.54mm_Vertical_SMD, symbol 4ms_Connector:Pins_02x05_SMT
- removed P1: Pins_02x05_TH, 4ms_Connector:Pins_2x05_2.54mm_TH, symbol 4ms_Connector:Pins_02x05_TH
- removed R16: 68k_0805, 4ms_Resistor:R_0805, symbol 4ms_Resistor:68k_0805
- removed R17, R22, R25: 100k_0805, 4ms_Resistor:R_Axial_DIN0207_L6.3mm_D2.5mm_P7.62mm_Horizontal, symbol 4ms_Resistor_TH:100k_TH0.125
- removed R24: 1M_0805, 4ms_Resistor:R_0805, symbol 4ms_Resistor:1M_0805
- removed R48, R49: 4.7k_0805, 4ms_Resistor:R_0805, symbol 4ms_Resistor_0805:4.7k_0805
- removed R6: 10k_0805, 4ms_Resistor:R_0805, symbol 4ms_Resistor:10k_0805
- removed R9: 1k_0805, 4ms_Resistor:R_Axial_DIN0207_L6.3mm_D2.5mm_P7.62mm_Horizontal, symbol 4ms_Resistor_TH:1k_TH0.125
- removed R?: 715, 4ms-footprints:R0603, symbol TrigSampler-rescue:R
- removed R?: 1.5k, 4ms-footprints:R0603, symbol TrigSampler-rescue:R
- removed R?: 7.15k, 4ms-footprints:R0603, symbol TrigSampler-rescue:R
- removed R?: 1.2k, 4ms-footprints:R0603, symbol TrigSampler-rescue:R
- removed R?: 7.87k, 4ms-footprints:R0603, symbol TrigSampler-rescue:R
- removed R?: 1k, 4ms-footprints:R0603, symbol TrigSampler-rescue:R
- removed R?: 2.7k, 4ms-footprints:R0603, symbol TrigSampler-rescue:R
- removed U13: PCA9685, 4ms-footprints:TSSOP-28_4.4x9.7mm_Pitch0.65mm, symbol TrigSampler-rescue:PCA9685
- removed U4: CONN_02X10, 4ms-footprints:CONN-2x10-SMT-127, symbol TrigSampler-rescue:Conn_02X10
- added C11: 100pF_Disc_TH, 4ms_Capacitor:C_Disc_P5.08mm, symbol 4ms_Capacitor:100pF_Disc_TH
- added C4, C5: 47uF_16V_TH, 4ms_Capacitor:CP_Radial_P2.5mm, symbol 4ms_Capacitor:47uF_16V_TH
- added C7, C8: 0.1uF_Disc_TH, 4ms_Capacitor:C_Disc_P2.54mm, symbol 4ms_Capacitor:0.1uF_Disc_TH
- added D1, D2: SB140-E3_TH, 4ms_Diode:D_DO-35_P7.62mm_Horizontal, symbol 4ms_Diode:SB140-E3_TH
- added J10, J11, J12, J8, J9: 3.5mm_Mono_Switched, 4ms_Jack:EighthInch_PJ398SM, symbol 4ms_Jack:3.5mm_Mono_Switched
- added J5: Eurorack_Power_16pin_Unshrouded, 4ms_Connector:Pins_2x08_2.54mm_TH_EuroPower, symbol 4ms_Connector:Eurorack_Power_16pin_Unshrouded
- added JA1, JB1, JC1, JD1: Socket_02x05_TH, 4ms_Connector:Socket_2x05_2.54mm_TH, symbol 4ms_Connector:Socket_02x05_TH
- added R12: 10k_TH0.125, 4ms_Resistor:R_Axial_DIN0204_L3.6mm_D1.6mm_P5.08mm_Horizontal, symbol 4ms_Resistor_TH:10k_TH0.125
- added R13: 68k_TH0.125, 4ms_Resistor:R_Axial_DIN0204_L3.6mm_D1.6mm_P5.08mm_Horizontal, symbol 4ms_Resistor_TH:68k_TH0.125
- added R14: 100k_TH0.125, 4ms_Resistor:R_Axial_DIN0204_L3.6mm_D1.6mm_P5.08mm_Horizontal, symbol 4ms_Resistor_TH:100k_TH0.125
- added R15: 1k_TH0.125, 4ms_Resistor:R_Axial_DIN0204_L3.6mm_D1.6mm_P5.08mm_Horizontal, symbol 4ms_Resistor_TH:1k_TH0.125
- added unit 2 of U2
- C1: renamed from C19; footprint 4ms_Capacitor:C_0805 -> 4ms_Capacitor:C_Disc_P2.54mm; symbol 4ms_Capacitor:1uF_0805_25V -> 4ms_Capacitor:0.1uF_Disc_TH; Display 1uF/25V -> 0.1uF
- C10: renamed from C23; footprint 4ms_Capacitor:C_0805 -> 4ms_Capacitor:C_Disc_P2.54mm; symbol 4ms_Capacitor:1uF_0805_25V -> 4ms_Capacitor:0.1uF_Disc_TH; Display 1uF/25V -> 0.1uF
- C2: renamed from C21; footprint 4ms_Capacitor:C_0805 -> 4ms_Capacitor:C_Disc_P2.54mm; symbol 4ms_Capacitor:1uF_0805_25V -> 4ms_Capacitor:0.1uF_Disc_TH; Display 1uF/25V -> 0.1uF
- C9: renamed from C20; footprint 4ms_Capacitor:C_0805 -> 4ms_Capacitor:C_Disc_P2.54mm; symbol 4ms_Capacitor:1uF_0805_25V -> 4ms_Capacitor:0.1uF_Disc_TH; Display 1uF/25V -> 0.1uF
- R10: renamed from R15; footprint 4ms_Resistor:R_0805 -> 4ms_Resistor:R_Axial_DIN0207_L6.3mm_D2.5mm_P7.62mm_Horizontal; symbol 4ms_Resistor_0805:33k_0805 -> 4ms_Resistor_TH:33k_TH0.125; Manufacturer Yageo -> Xicon; Part Number RC0805FR-0733KL -> 299-33k-RC; Specifications 33k, 1%, 1/8W, 0805 -> 33k, 5%, 1/8W, TH0.125
- R17: renamed from R38; footprint 4ms_Resistor:R_0805 -> 4ms_Resistor:R_Axial_DIN0207_L6.3mm_D2.5mm_P7.62mm_Horizontal; symbol 4ms_Resistor_0805:2.7k_0805 -> 4ms_Resistor_TH:2.7k_TH0.125; Manufacturer Yageo -> Xicon; Part Number RC0805FR-072K7L -> 299-2.7k-RC; Specifications 2.7k, 1%, 1/8W, 0805 -> 2.7k, 5%, 1/8W, TH0.125
- R18: renamed from R44; footprint 4ms-footprints:R0603 -> 4ms_Resistor:R_Axial_DIN0207_L6.3mm_D2.5mm_P7.62mm_Horizontal; symbol TrigSampler-rescue:R -> 4ms_Resistor_TH:150Ω_TH0.125; Display (none) -> 150Ω; Manufacturer (none) -> Xicon; Part Number (none) -> 299-150-RC; Specifications (none) -> 150Ω, 5%, 1/8W, TH0.125
- R19: renamed from R46; footprint 4ms-footprints:R0603 -> 4ms_Resistor:R_Axial_DIN0207_L6.3mm_D2.5mm_P7.62mm_Horizontal; symbol TrigSampler-rescue:R -> 4ms_Resistor_TH:150Ω_TH0.125; Display (none) -> 150Ω; Manufacturer (none) -> Xicon; Part Number (none) -> 299-150-RC; Specifications (none) -> 150Ω, 5%, 1/8W, TH0.125
- R21: renamed from R33; footprint 4ms_Resistor:R_0805 -> 4ms_Resistor:R_Axial_DIN0207_L6.3mm_D2.5mm_P7.62mm_Horizontal; symbol 4ms_Resistor_0805:2.7k_0805 -> 4ms_Resistor_TH:2.7k_TH0.125; Manufacturer Yageo -> Xicon; Part Number RC0805FR-072K7L -> 299-2.7k-RC; Specifications 2.7k, 1%, 1/8W, 0805 -> 2.7k, 5%, 1/8W, TH0.125
- R23: renamed from R47; footprint 4ms-footprints:R0603 -> 4ms_Resistor:R_Axial_DIN0207_L6.3mm_D2.5mm_P7.62mm_Horizontal; symbol TrigSampler-rescue:R -> 4ms_Resistor_TH:150Ω_TH0.125; Display (none) -> 150Ω; Manufacturer (none) -> Xicon; Part Number (none) -> 299-150-RC; Specifications (none) -> 150Ω, 5%, 1/8W, TH0.125
- R25: renamed from R35; footprint 4ms_Resistor:R_0805 -> 4ms_Resistor:R_Axial_DIN0207_L6.3mm_D2.5mm_P7.62mm_Horizontal; symbol 4ms_Resistor_0805:4.7k_0805 -> 4ms_Resistor_TH:4.7k_TH0.125; Manufacturer Yageo -> Xicon; Part Number RC0805FR-074K7L -> 299-4.7k-RC; Specifications 4.7k, 1%, 1/8W, 0805 -> 4.7k, 5%, 1/8W, TH0.125
- R26: renamed from R43; footprint 4ms_Resistor:R_0805 -> 4ms_Resistor:R_Axial_DIN0207_L6.3mm_D2.5mm_P7.62mm_Horizontal; symbol 4ms_Resistor_0805:4.7k_0805 -> 4ms_Resistor_TH:4.7k_TH0.125; Manufacturer Yageo -> Xicon; Part Number RC0805FR-074K7L -> 299-4.7k-RC; Specifications 4.7k, 1%, 1/8W, 0805 -> 4.7k, 5%, 1/8W, TH0.125
- R27: renamed from R31; footprint 4ms_Resistor:R_0805 -> 4ms_Resistor:R_Axial_DIN0207_L6.3mm_D2.5mm_P7.62mm_Horizontal; symbol 4ms_Resistor_0805:4.7k_0805 -> 4ms_Resistor_TH:4.7k_TH0.125; Manufacturer Yageo -> Xicon; Part Number RC0805FR-074K7L -> 299-4.7k-RC; Specifications 4.7k, 1%, 1/8W, 0805 -> 4.7k, 5%, 1/8W, TH0.125
- R28: renamed from R10; footprint 4ms_Resistor:R_0805 -> 4ms_Resistor:R_Axial_DIN0207_L6.3mm_D2.5mm_P7.62mm_Horizontal; symbol 4ms_Resistor_0805:33k_0805 -> 4ms_Resistor_TH:33k_TH0.125; Manufacturer Yageo -> Xicon; Part Number RC0805FR-0733KL -> 299-33k-RC; Specifications 33k, 1%, 1/8W, 0805 -> 33k, 5%, 1/8W, TH0.125
- R29: renamed from R11; footprint 4ms_Resistor:R_0805 -> 4ms_Resistor:R_Axial_DIN0207_L6.3mm_D2.5mm_P7.62mm_Horizontal; symbol 4ms_Resistor_0805:33k_0805 -> 4ms_Resistor_TH:33k_TH0.125; Manufacturer Yageo -> Xicon; Part Number RC0805FR-0733KL -> 299-33k-RC; Specifications 33k, 1%, 1/8W, 0805 -> 33k, 5%, 1/8W, TH0.125
- R30: renamed from R12; footprint 4ms_Resistor:R_0805 -> 4ms_Resistor:R_Axial_DIN0207_L6.3mm_D2.5mm_P7.62mm_Horizontal; symbol 4ms_Resistor_0805:33k_0805 -> 4ms_Resistor_TH:33k_TH0.125; Manufacturer Yageo -> Xicon; Part Number RC0805FR-0733KL -> 299-33k-RC; Specifications 33k, 1%, 1/8W, 0805 -> 33k, 5%, 1/8W, TH0.125
- R31: renamed from R13; footprint 4ms_Resistor:R_0805 -> 4ms_Resistor:R_Axial_DIN0207_L6.3mm_D2.5mm_P7.62mm_Horizontal; symbol 4ms_Resistor_0805:33k_0805 -> 4ms_Resistor_TH:33k_TH0.125; Manufacturer Yageo -> Xicon; Part Number RC0805FR-0733KL -> 299-33k-RC; Specifications 33k, 1%, 1/8W, 0805 -> 33k, 5%, 1/8W, TH0.125
- R32: renamed from R14; footprint 4ms_Resistor:R_0805 -> 4ms_Resistor:R_Axial_DIN0207_L6.3mm_D2.5mm_P7.62mm_Horizontal; symbol 4ms_Resistor_0805:33k_0805 -> 4ms_Resistor_TH:33k_TH0.125; Manufacturer Yageo -> Xicon; Part Number RC0805FR-0733KL -> 299-33k-RC; Specifications 33k, 1%, 1/8W, 0805 -> 33k, 5%, 1/8W, TH0.125
- U6: renamed from U11; footprint 4ms-footprints:LED-3MM-SQUARE-ANODE -> 4ms_LED:LED_3mm_C1A2_Polarity_Indicator
- renumbered C13 to C12, C14 to C13, C15 to C14, C16 to C15, C29 to C16, C31 to C17, C26 to C18, C1 to C3, C5 to C6, J4 to J2, J5 to J3, J2 to J4, J7 to J6, J6 to J7, U6 to POT_LENGTH1, U5 to POT_PITCH1, U7 to POT_SAMPLE1, U9 to POT_STARTPOS1, R4 to R1, R2 to R11, R36 to R16, R3 to R2, R32 to R20, R39 to R22, R34 to R24, R18 to R3, R29 to R33, R19 to R4, R7 to R5, R20 to R6, R21 to R7, R1 to R9, S2 to S1, S4 to S2, S1 to S3, IC2 to U1, IC1 to U2
Connections:
- net +3.3VADC is gone; now on net VREF+: POT_LENGTH1.3 (Right), POT_PITCH1.3 (Right), POT_SAMPLE1.3 (Right), POT_STARTPOS1.3 (Right)
- net BANK1_B_LED is gone; now on net D8: R22.2
- net BANK1_G_LED is gone; now on net D5: R16.1
- net BANK1_R_LED is gone; now on net D6: R17.1
- net PLAY1_B_LED is gone; now on net D14: R23.2
- net PLAY1_G_LED is gone; now on net D7: R18.1
- net PLAY1_LED is gone; now on net D12: U6.2 (A)
- net PLAY1_R_LED is gone; now on net D3: R19.1
- net SDIO_CLK is gone; now on net D9: CON1.5 (CLK)
- net SDIO_CMD is gone; now on net D19: CON1.3 (CMD), R30.2
- net SDIO_D0 is gone; now on net D16: CON1.7 (DAT0), R31.2
- net SDIO_D1 is gone; now on net D17: CON1.8 (DAT1), R32.2
- net SDIO_D2 is gone; now on net D18: CON1.1 (DAT2), R28.2
- net +12V: now also C4.1, C7.1, D1.1 (K), JA1.9 (-12V)
- net +3V3: now also JD1.8 (GND)
- net -12VA: now also C5.2, C8.1, D2.2 (A), JA1.1 (+12V)
- net A0: now also JC1.1 (+12V)
- net A1: now also JC1.2 (+12V)
- net A2: now also JC1.3 (GND)
- net A3: now also JC1.4 (GND)
- net A4: now also JC1.5 (GND)
- net A5: now also JC1.6 (GND)
- net A6: now also JC1.7 (GND)
- net A7: now also JC1.8 (GND)
- net A8: now also JC1.9 (-12V)
- net A9: now also JC1.10 (-12V)
- net D0: now also JB1.2 (+12V)
- net D1: now also J7.1 (SIG), JB1.4 (GND)
- net D10: now also JA1.4 (GND)
- net D11: now also C17.1, R26.2, JA1.3 (GND)
- net D12: now also JA1.6 (GND); no longer C17.1, R26.2
- net D13: now also JB1.8 (GND); no longer C18.1, R27.2
- net D14: now also JA1.5 (GND)
- net D15: now also JB1.6 (GND)
- net D16: now also JD1.9 (-12V)
- net D17: now also JD1.7 (GND)
- net D18: now also JD1.5 (GND)
- net D19: now also JD1.3 (GND)
- net D2: now also JB1.10 (-12V), R12.1
- net D3: now also JB1.9 (-12V)
- net D5: now also JD1.1 (+12V)
- net D6: now also JD1.2 (+12V)
- net D7: now also JD1.6 (GND)
- net D8: now also JD1.4 (GND)
- net D9: now also JD1.10 (-12V)
- net GND: now also C4.2, C5.1, C7.2, C8.2, J10.2 (SHEILD), J11.2 (SHEILD), J12.2 (SHEILD), J5.10 (GND), J5.11 (GND), J5.12 (GND), J5.13 (-12), J5.14 (-12V), J5.9 (GND), J8.2 (SHEILD), J9.2 (SHEILD), JA1.7 (GND), R13.1
- net GNDADC: now also JA1.8 (GND)
- net Unused(5V): now also JA1.10 (-12V)
- net VREF+: now also JA1.2 (+12V)
- net REV1_B_LED: no longer names the net of R24.2
- net REV1_G_LED: no longer names the net of R20.1
- net REV1_R_LED: no longer names the net of R21.1
- net SDIO_D3: no longer names the net of CON1.2 (CD/DAT3), R29.2
- new net: C11.2, R14.2, R15.1, U2.7
- new net: J10.1 (SIG), R15.2
- new net: C11.1, R13.2, R14.1, U2.6 (-)
- new net: D2.1 (K), J5.15 (-12V), J5.16 (P16)
- new net: D1.2 (A), J5.7 (12V), J5.8 (+12V)
- new net: R12.2, U2.5 (+)
- new net: C18.1, R27.2
- new net AUDIO_IN1: J12.1 (SIG), JB1.7 (GND)
- new net AUDIO_IN2: J8.1 (SIG), JB1.5 (GND)
- new net AUDIO_OUT1: J9.1 (SIG), JB1.3 (GND)
- new net AUDIO_OUT2: J11.1 (SIG), JB1.1 (+12V)
- new net PWR_HDR_CLK_BUS: J5.1 (P1), J5.2 (P2)
- no-connect marks 20 -> 15
Other:
- note added: "4ms STS Kit"
- note added: "Audio"
- note added: "Bank_But_B"
- note added: "Bank_But_G"
- note added: "Bank_But_R"
- note added: "Buttons/Switches"
- note added: "Headers"
- note added: "LED"
- note added: "PLAY_LED"
- note added: "POWER"
- note added: "Play_But_B"
- note added: "Play_But_G"
- note added: "Play_But_R"
- note added: "Pots"
- note added: "Rev_But_B"
- note added: "Rev_But_G"
- note added: "Rev_But_R"
- note added: "SD CARD"
- note added: "SD Card"
- note added: "need to double-check the pins used for those LEDs have a TIM PWM channel output on cubemx. digital pins for this have not yet been assigned"
- note removed: "(5V)"
- note removed: "(TDI)"
- note removed: "12C1_SCL"
- note removed: "12C2_SDA"
- note removed: "I am not sure which of the multi-use pins we are gonna need if any, I assigned the digital pins arbitrarily for the time being."
- note removed: "I'll update the LED labels once I get the PCA question figured out"
- note removed: "Like this?? I was looking at the DLD Kit and it made me wonder about part B of Jack 1"
- note removed: "Rec_But"
- note removed: "Rec_Trig"
- note removed: "SPI5_MISO"
- note removed: "SPI5_MOSI"
- note removed: "SPI5_NSS"
- note removed: "SPI5_SCK"
- note removed: "Trace pins are generic Digital pins? Needs updating I was not sure what to do with this."
- note removed: "We don't have a library part for socket. The Samtec part number associated with these headers is for pins, update this."
- note removed: "double check this, I chose D16 arbitrarily for time being"
- moved on the sheet: C1, C10, C12, C13, C14, C15, C16, C17, C18, C2, C9, CON1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

Commit message: part placement
Parts:
- removed R33: 1k_0805, 4ms_Resistor:R_Axial_DIN0207_L6.3mm_D2.5mm_P7.62mm_Horizontal, symbol 4ms_Resistor_TH:1k_TH0.125
- removed S2: Button_SPST_RGB_5.4mmCap, 4ms_Switch:Button_RgbLED_SPST_PB615303HL-7mm, symbol 4ms_Switch:Button_SPST_RGB_5.4mmCap
- removed U6: white, 4ms_LED:LED_3mm_C1A2_Polarity_Indicator, symbol TrigSampler-rescue:LED-RESCUE-TrigSampler
- added PLAY_BUT1: Button_SPST_RGB_7mmCap, 4ms_Switch:Button_RgbLED_SPST_PB615303HL-7mm, symbol 4ms_Switch:Button_SPST_RGB_7mmCap
- C1, C10, C2, C9: value 1uF_0805_25V -> 0.1uF_Disc_TH; Manufacturer Murata -> (none); Part Number GCM219R91H103KA37D -> (none); Specifications 1uF, 25V, 0805, MLCC, X5R or similar -> (none)
- C12, C13, C14, C15, C16, C17, C18, C3: value 0.1uF_0805_50V -> 0.1uF_Disc_TH; Manufacturer Murata -> (none); Part Number GCJ21BL81H104KA01L -> (none); Specifications 0.1uF, 50V, 0805, MLCC, X5R or similar -> (none)
- C6: value 1nF_0603_50V -> 1nF_Disc_TH; symbol 4ms_Capacitor:1nF_0603_50V -> 4ms_Capacitor:1nF_Disc_TH
- J1: value 3.5mm_Mono_Switched -> START_CV
- J10: renamed from J12; value 3.5mm_Mono_Switched -> AUDIO_INR
- J11: value 3.5mm_Mono_Switched -> AUDIO_OUTL
- J2: value 3.5mm_Mono_Switched -> LENGTH_CV
- J3: value 3.5mm_Mono_Switched -> SAMP_CV
- J4: value 3.5mm_Mono_Switched -> PITCH CV
- J5: renamed from J6; value 3.5mm_Mono_Switched -> REV_TRIG
- J6: renamed from J7; value 3.5mm_Mono_Switched -> PLAY_TRIG
- J7: renamed from J10; value 3.5mm_Mono_Switched -> END_OUT
- J8: value 3.5mm_Mono_Switched -> AUDIO_INL
- J9: value 3.5mm_Mono_Switched -> AUIDO_OUTR
- R1, R11, R16, R20, R22, R24: value 1k_0805 -> 1k_TH0.125
- R10, R28, R29, R30, R31, R32: value 33k_0805 -> 33k_TH0.125; JLCPCB ID C141696 -> (none)
- R12, R13, R14, R15: footprint 4ms_Resistor:R_Axial_DIN0204_L3.6mm_D1.6mm_P5.08mm_Horizontal -> 4ms_Resistor:R_Axial_DIN0207_L6.3mm_D2.5mm_P7.62mm_Horizontal
- R17, R21: value 2.7k_0805 -> 2.7k_TH0.125; JLCPCB ID C114520 -> (none)
- R18, R19, R23: value 150 -> 150Ω_TH0.125
- R2, R3, R4: value 49.9k_0805 -> 47k_TH0.125; JLCPCB ID C114540 -> (none)
- R25, R26, R27: value 4.7k_0805 -> 4.7k_TH0.125; JLCPCB ID C60816 -> (none)
- R5, R6, R7, R8: value 100k_0805 -> 100k_TH0.125; JLCPCB ID C96346 -> (none)
- R9: value 620 -> 620Ω_TH0.125
- U1: renamed from U2; value TL082 -> TL082_TH; JLCPCB ID C2652280 -> (none); Manufacturer STMicroelectronics -> (none); Part Number TL082CPT -> (none)
- U1, U2: value TL082 -> TL082_TH; JLCPCB ID C2652280 -> (none); Manufacturer STMicroelectronics -> (none); Part Number TL082CPT -> (none)
- U2: renamed from U1; value TL082 -> TL082_TH; JLCPCB ID C2652280 -> (none); Manufacturer STMicroelectronics -> (none); Part Number TL082CPT -> (none)
- renumbered S1 to BANK_BUT1, J5 to J12, POT_SAMPLE1 to POT_SAMP1, POT_STARTPOS1 to POT_START1, S3 to REV_BUT1, CON1 to SD1
Connections:
- net +3V3: now also PLAY_BUT1.5 (CA)
- net A9: now also C18.1, R27.2
- net D0: now also R22.2; no longer J5.1 (SIG)
- net D1: now also R17.1; no longer J6.1 (SIG)
- net D10: now also R20.1; no longer C16.1, R25.2
- net D11: now also R24.2; no longer C17.1, R26.2
- net D12: now also R21.1
- net D13: now also J6.1 (SIG)
- net D15: now also J5.1 (SIG)
- net D6: now also C16.1, R25.2; no longer R17.1
- net D8: now also C17.1, R26.2; no longer R22.2
- net GND: now also PLAY_BUT1.4 (UP-B)
- net at R18.2: now also PLAY_BUT1.8 (B)
- net at R26.1: now also PLAY_BUT1.2 (POLE-A)
- net at R23.1: now also PLAY_BUT1.6 (G)
- net at R19.2: now also PLAY_BUT1.7 (R)
Other:
- note added: "*"
- note added: "* = No PWM"
- note removed: "LED"
- note removed: "PLAY_LED"
- note removed: "need to double-check the pins used for those LEDs have a TIM PWM channel output on cubemx. digital pins for this have not yet been assigned"
