File: faceplate/p2-smt/Kit-Trig-Sampler-FACEPLATE.kicad_pcb (KiCad board)
At the start: 2 copper layers, 80.9 x 128.5 mm, 24 parts

Commit message: p3 smt: redid faceplate
Parts:
- added ?: , , F.Cu at (51.1, 7.37)
- added REF**: Rail_Connection_16HP, 4ms_Faceplate:Rail_Connection_16HP, B.Cu at (50.8, 126.7)
