File: p3/Kit-Trig-Sampler.kicad_sch (KiCad schematic)
At the start: 92 parts, among them J1 3.5mm_Mono_Switched, J10 3.5mm_Mono_Switched, J11 3.5mm_Mono_Switched, J13 3.5mm_Mono_Switched, J14 Eurorack_Power_10pin_Unshroud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, J2 3.5mm_Mono_Switched, J3 3.5mm_Mono_Switched, J4 3.5mm_Mono_Switched, J5 3.5mm_Mono_Switched, J6 3.5mm_Mono_Switched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

Commit message: finish p3-SMT BOM. Update all headers to non-gold
Parts:
- JA1, JB1, JC1, JD1: Part Number SSW-105-01-G-D -> SSW-105-01-T-D; Specifications HEADER 2x5 FEMALE SOCKET 0.100” 180deg -> HEADER 2x5 FEMALE SOCKET 0.100” 180deg, Height=8.5mm
- KNOB1, KNOB2, KNOB3, KNOB4: Specifications White Line, Diameter: ?mm, D-shaft 3.5mm depth -> D-shaft, 3.5mm depth
Changed lines of the file:
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@@
       (effects (font (size 1.27 1.27)) hide)
     )
-    (property "Specifications" "HEADER 2x5 FEMALE SOCKET 0.100” 180deg" (at 478.79 228.6 0)
+    (property "Specifications" "HEADER 2x5 FEMALE SOCKET 0.100” 180deg, Height=8.5mm" (at 478.79 228.6 0)
       (effects (font (size 1.27 1.27)) (justify left) hide)
     )
@@
       (effects (font (size 1.27 1.27)) (justify left) hide)
     )
-    (property "Part Number" "SSW-105-01-G-D" (at 478.79 223.52 0)
+    (property "Part Number" "SSW-105-01-T-D" (at 478.79 223.52 0)
       (effects (font (size 1.27 1.27)) (justify left) hide)
     )
@@
       (effects (font (size 1.27 1.27)) hide)
     )
-    (property "Specifications" "HEADER 2x5 FEMALE SOCKET 0.100” 180deg" (at 478.79 260.35 0)
+    (property "Specifications" "HEADER 2x5 FEMALE SOCKET 0.100” 180deg, Height=8.5mm" (at 478.79 260.35 0)
       (effects (font (size 1.27 1.27)) (justify left) hide)
     )
@@
       (effects (font (size 1.27 1.27)) (justify left) hide)
     )
-    (property "Part Number" "SSW-105-01-G-D" (at 478.79 255.27 0)
+    (property "Part Number" "SSW-105-01-T-D" (at 478.79 255.27 0)
       (effects (font (size 1.27 1.27)) (justify left) hide)
     )
@@
   )
   (symbol (lib_id "4ms_Hardware:Knob_Davies_WhiteLine") (at 452.12 387.35 0) (unit 1)
-    (in_bom yes) (on_board no) (dnp no) (fields_autoplaced)
+    (in_bom yes) (on_board yes) (dnp no) (fields_autoplaced)
     (property "Reference" "KNOB3" (at 457.2 387.985 0)
       (effects (font (size 1.27 1.27)) (justify left))
@@
       (effects (font (size 1.27 1.27)) hide)
     )
-    (property "Specifications" "White Line, Diameter: ?mm, D-shaft 3.5mm depth" (at 452.12 394.97 0)
+    (property "Specifications" "D-shaft, 3.5mm depth" (at 452.12 394.97 0)
       (effects (font (size 1.27 1.27)) hide)
     )
@@
   )
   (symbol (lib_id "4ms_Hardware:Knob_Davies_WhiteLine") (at 435.61 400.05 0) (unit 1)
-    (in_bom yes) (on_board no) (dnp no) (fields_autoplaced)
+    (in_bom yes) (on_board yes) (dnp no) (fields_autoplaced)
     (property "Reference" "KNOB2" (at 440.69 400.685 0)
       (effects (font (size 1.27 1.27)) (justify left))
@@
       (effects (font (size 1.27 1.27)) hide)
     )
-    (property "Specifications" "White Line, Diameter: ?mm, D-shaft 3.5mm depth" (at 435.61 407.67 0)
+    (property "Specifications" "D-shaft, 3.5mm depth" (at 435.61 407.67 0)
       (effects (font (size 1.27 1.27)) hide)
     )
@@
       (effects (font (size 1.27 1.27)) hide)
     )
-    (property "Specifications" "HEADER 2x5 FEMALE SOCKET 0.100” 180deg" (at 386.08 260.35 0)
+    (property "Specifications" "HEADER 2x5 FEMALE SOCKET 0.100” 180deg, Height=8.5mm" (at 386.08 260.35 0)
       (effects (font (size 1.27 1.27)) (justify left) hide)
     )
@@
       (effects (font (size 1.27 1.27)) (justify left) hide)
     )
-    (property "Part Number" "SSW-105-01-G-D" (at 386.08 255.27 0)
+    (property "Part Number" "SSW-105-01-T-D" (at 386.08 255.27 0)
       (effects (font (size 1.27 1.27)) (justify left) hide)
     )
@@
   )
   (symbol (lib_id "4ms_Hardware:Knob_Davies_WhiteLine") (at 452.12 400.05 0) (unit 1)
-    (in_bom yes) (on_board no) (dnp no) (fields_autoplaced)
+    (in_bom yes) (on_board yes) (dnp no) (fields_autoplaced)
     (property "Reference" "KNOB4" (at 457.2 400.685 0)
       (effects (font (size 1.27 1.27)) (justify left))
@@
       (effects (font (size 1.27 1.27)) hide)
     )
-    (property "Specifications" "White Line, Diameter: ?mm, D-shaft 3.5mm depth" (at 452.12 407.67 0)
+    (property "Specifications" "D-shaft, 3.5mm depth" (at 452.12 407.67 0)
       (effects (font (size 1.27 1.27)) hide)
     )
@@
       (effects (font (size 1.27 1.27)) hide)
     )
-    (property "Specifications" "HEADER 2x5 FEMALE SOCKET 0.100” 180deg" (at 386.08 227.33 0)
+    (property "Specifications" "HEADER 2x5 FEMALE SOCKET 0.100” 180deg, Height=8.5mm" (at 386.08 227.33 0)
       (effects (font (size 1.27 1.27)) (justify left) hide)
     )
@@
       (effects (font (size 1.27 1.27)) (justify left) hide)
     )
-    (property "Part Number" "SSW-105-01-G-D" (at 386.08 222.25 0)
+    (property "Part Number" "SSW-105-01-T-D" (at 386.08 222.25 0)
       (effects (font (size 1.27 1.27)) (justify left) hide)
     )
@@
   )
   (symbol (lib_id "4ms_Hardware:Knob_Davies_WhiteLine") (at 435.61 387.35 0) (unit 1)
-    (in_bom yes) (on_board no) (dnp no) (fields_autoplaced)
+    (in_bom yes) (on_board yes) (dnp no) (fields_autoplaced)
     (property "Reference" "KNOB1" (at 440.69 387.985 0)
       (effects (font (size 1.27 1.27)) (justify left))
@@
       (effects (font (size 1.27 1.27)) hide)
     )
-    (property "Specifications" "White Line, Diameter: ?mm, D-shaft 3.5mm depth" (at 435.61 394.97 0)
+    (property "Specifications" "D-shaft, 3.5mm depth" (at 435.61 394.97 0)
       (effects (font (size 1.27 1.27)) hide)
     )
