File: v1.0-kit/Kit-Trig-Sampler.kicad_sch (KiCad schematic)
At the start: 92 parts, among them J1 3.5mm_Mono_Switched, J10 3.5mm_Mono_Switched, J11 3.5mm_Mono_Switched, J13 3.5mm_Mono_Switched, J14 Eurorack_Power_10pin_Unshroud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, J2 3.5mm_Mono_Switched, J3 3.5mm_Mono_Switched, J4 3.5mm_Mono_Switched, J5 3.5mm_Mono_Switched, J6 3.5mm_Mono_Switched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

Commit message: v1.0-kit: updated BOM (new TH part numbers to match what we actually use)
Parts:
- C1, C10, C12, C13, C14, C15, C16, C17, C2, C3, C7, C8, C9: Part Number K104Z15Y5VF53L2 -> K104K15X7RF5TL2; Specifications MLCC, Leaded, Min 25V, Y5V, Lead Spacing 2.5mm, Body approx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 -> MLCC, Leaded, Min 25V, Y5V or X7R, Lead Spacing 2.5mm, Body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
- C19, C20, C4, C5: Manufacturer Panasonic -> Kemet; Manufacturer 2 Lelon -> Kemet; Part Number ECA-1VM470I -> ESW476M035AE3AA; Part Number 2 RGA470M1VBK-0611G -> ESY476M050AE3AA; Specifications Aluminum Electrolytic, Radial Leaded, Min 25V, 5mm Diameter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 -> Aluminum Electrolytic, Radial Leaded, Min 16V, 6.3mm Diamet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
