File: v1.1-rc-1_12HP/Sampler-built.kicad_sch (KiCad schematic)
At the start: 238 parts, among them J10 Eurorack_Power_10pin_Unshroud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, J11 3.5mm_Mono_Switched, J12 3.5mm_Mono_Switched, J13 3.5mm_Mono_Switched, J14 3.5mm_Mono_Switched, J15 3.5mm_Mono_Switched, J16 3.5mm_Mono_Switched, J17 3.5mm_Mono_Switched, J2 3.5mm_Mono_Switched, J3 Conn_01x04, J4 Conn_02x04, J6 3.5mm_Mono_Switched, J7 3.5mm_Mono_Switched, J8 3.5mm_Mono_Switched, J9 3.5mm_Mono_Switched, U1 TL072H, U10 TL072H, U11 TL072H, U12 TL072H, U13 AP62200WU-7, U14 TL072H, U15 NJM2068, U16 NJM2068, U18 STS SD card w/adaptor, U2 STM32F746IE, U3 TL072H, U4 SDRAM_IS42S16400J-6BLI-TR, U5 TL072H, U6 NCP51460SN33, U8 TL072H, U9 PCM3060PW, Y1 16MHz_18pF_FA238

Commit message: SCH: Updated STM chip (U2) to use new library part.
Set kicad.sch file back to v7
Parts:
- FP1: Part Number sampler-faceplate-v1.0 -> (none); Production Stage D -> F; Specifications Sampler Faceplate, FR-4, HASL-LF, matte black mask, white s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 -> (none)
- NT1, NT2: footprint NetTie:NetTie-2_SMD_Pad0.5mm -> (none)
- PCB1: Part Number sampler-v1.0 -> (none); Production Stage D -> F; Specifications matte black mask, white silk, FR4 1.6mm, HASL-LF, two layer -> (none)
- U2: symbol 4ms_IC:STM32F730I8 -> 4ms_IC:STM32F746IE; Part Number STM32F746IEK6 -> STM32F746IE; Specifications ARM Cortex-M7, KB flash, 256KB RAM, 216MHz, UFBGA-176 -> ARM Cortex-M7, 64KB flash, 256KB RAM, 216MHz, UFBGA-176
- V1: JLCPCB ID (none) -> C50754; JLCPCB ID 2 (none) -> C512090; JLCPCB ID 3 (none) -> C625398

Commit message: SCH: Replaced NJMs with 072Hs - PCB: updated PCB from schematic
Parts:
- U15, U16: value NJM2068 -> TL072H; symbol 4ms_IC:NJM2068 -> 4ms_IC:TL072H; JLCPCB ID (none) -> C4370341; Manufacturer NJR -> Texas Instruments; Part Number NJM2068V-TE1 -> TL072HIPWR; Specifications NJM2068 Dual Opamp -> Dual Opamp TSSOP-8

Commit message: TODO for v1.1-rc2 (12HP)
Other:
- note added: "TODO for v1.1rc2: - SD Card is rotated 180 degrees (compared to STS and kit Sampler) - Pot and CV ADC pins are not the same as kit version (swapped Length and Start Pos pots? swapped Bank and Sample CV??) - Left and Right outputs are swapped on kit version, so we should do the same here - Pressing REV shorts it out?"
Changed lines of the file:
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@@
     (effects (font (size 1.27 1.27)) (justify right bottom))
+  )
+  (text "TODO for v1.1rc2:\n- SD Card is rotated 180 degrees (compared to STS and kit Sampler)\n- Pot and CV ADC pins are not the same as kit version (swapped Length and Start Pos pots?\nswapped Bank and Sample CV??)\n- Left and Right outputs are swapped on kit version, so we should do the same here\n- Pressing REV shorts it out?"
+    (at 582.93 278.13 0)
+    (effects (font (size 4 4)) (justify left bottom))
   )
   (text "Buttons/Switches" (at 725.17 44.45 0)
