File: v1.1-rc-1_12HP/Sampler-built.kicad_sch (KiCad schematic)
At the start: 238 parts, among them J10 Eurorack_Power_10pin_Unshroud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, J11 3.5mm_Mono_Switched, J12 3.5mm_Mono_Switched, J13 3.5mm_Mono_Switched, J14 3.5mm_Mono_Switched, J15 3.5mm_Mono_Switched, J16 3.5mm_Mono_Switched, J17 3.5mm_Mono_Switched, J2 3.5mm_Mono_Switched, J3 Conn_01x04, J4 Conn_02x04, J6 3.5mm_Mono_Switched, J7 3.5mm_Mono_Switched, J8 3.5mm_Mono_Switched, J9 3.5mm_Mono_Switched, U1 TL072H, U10 TL072H, U11 TL072H, U12 TL072H, U13 AP62200WU-7, U14 TL072H, U15 TL072H, U16 TL072H, U18 STS SD card w/adaptor, U2 STM32F746IE, U3 TL072H, U4 SDRAM_IS42S16400J-6BLI-TR, U5 TL072H, U6 NCP51460SN33, U8 TL072H, U9 PCM3060PW, Y1 16MHz_18pF_FA238

Commit message: v1.1rc-1 was accidentally updated from how it was produced. Reverted the folder back to an earlier commit
Connections:
- net A3: now also R23.2; no longer R41.2
- net A4: now also R28.2; no longer R34.2
- net A7: now also R41.2; no longer R23.2
- net A8: now also R34.2; no longer R28.2
- net at J16.1 (SIG): now also R153.1; no longer R152.1
- net at J17.1 (SIG): now also R152.1; no longer R153.1
Other:
- note added: "TODO for v1.1rc2: - SD Card is rotated 180 degrees (compared to STS and kit Sampler) - Pot and CV ADC pins are not the same as kit version (swapped Length and Start Pos pots? swapped Bank and Sample CV??) - Left and Right outputs are swapped on kit version, so we should do the same here - Pressing REV shorts it out?"
- note removed: "TODO for v1.1rc2: - xSD Card is rotated 180 degrees (compared to STS and kit Sampler) - XPot and CV ADC pins are not the same as kit version (swapped Length and Start Pos pots? swapped Bank and Sample CV??) - SWAP LENGTH AND START POTS. SWAP BANK AND SAMP - XLeft and Right outputs are swapped on kit version, so we should do the same here - xPressing REV shorts it out?"
- moved on the sheet: J16, J17
