File: v1.1-rc-2_12HP/Sampler-built.kicad_sch (KiCad schematic)
At the start: 238 parts, among them J10 Eurorack_Power_10pin_Unshroud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, J11 3.5mm_Mono_Switched, J12 3.5mm_Mono_Switched, J13 3.5mm_Mono_Switched, J14 3.5mm_Mono_Switched, J15 3.5mm_Mono_Switched, J16 3.5mm_Mono_Switched, J17 3.5mm_Mono_Switched, J2 3.5mm_Mono_Switched, J3 Conn_01x04, J4 Conn_02x04, J6 3.5mm_Mono_Switched, J7 3.5mm_Mono_Switched, J8 3.5mm_Mono_Switched, J9 3.5mm_Mono_Switched, U1 TL072H, U10 TL072H, U11 TL072H, U12 TL072H, U13 AP62200WU-7, U14 TL072H, U15 TL072H, U16 TL072H, U18 STS SD card w/adaptor, U2 STM32F746IE, U3 TL072H, U4 SDRAM_IS42S16400J-6BLI-TR, U5 TL072H, U6 NCP51460SN33, U8 TL072H, U9 PCM3060PW, Y1 16MHz_18pF_FA238

Commit message: Updated todo list and added soft start circuit. Todo: add solder jumpers
Parts:
- added C? (x2): 100nF_0603_16V, 4ms_Capacitor:C_0603, symbol 4ms_Capacitor:100nF_0603_16V
- added Q?: Si2318, 4ms_Package_SOT:SOT23-3_PO132, symbol 4ms_Transistor:Si2318
- added Q?: Si2347, 4ms_Package_SOT:SOT23-3_PO132, symbol 4ms_Transistor:Si2347
- added R? (x2): 1M_0603, 4ms_Resistor:R_0603, symbol 4ms_Resistor_0603:1M_0603
Connections:
- net +12V: now also Q?.3 (D); no longer C25.1, D16.1 (K)
- net -12VA: now also Q?.3 (D); no longer C26.1, D17.2 (A)
- net GND: now also R?.1, R?.1
- new net: C?.2, Q?.1 (G), R?.2 (x2)
- new net: C26.1, C?.1, D17.2 (A), Q?.2 (S)
- new net: C25.1, C?.1, D16.1 (K), Q?.2 (S)
Other:
- note added: "TODO for v1.1rc2: [x] SD Card is rotated 180 degrees (compared to STS and kit Sampler) [x] Pot and CV ADC pins are not the same as kit version (swapped Length and Start Pos pots? swapped Bank and Sample CV??) - SWAP LENGTH AND START POTS. SWAP BANK AND SAMP [x] Left and Right outputs are swapped on kit version, so we should do the same here [x] Pressing REV shorts it out? [ ] Find out from Dan wh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"
- note removed: "TODO for v1.1rc2: - xSD Card is rotated 180 degrees (compared to STS and kit Sampler) - XPot and CV ADC pins are not the same as kit version (swapped Length and Start Pos pots? swapped Bank and Sample CV??) - SWAP LENGTH AND START POTS. SWAP BANK AND SAMP - XLeft and Right outputs are swapped on kit version, so we should do the same here - xPressing REV shorts it out?"
- note removed: "TODO: Consolidate CV op-amps based on where they are placed on PCB. Use a single opamp if needed (most likely for PitchCV)"
- moved on the sheet: C21, C24, C25, C26

Commit message: Added softstart to +/-12v rails - and solder jumpers between +12v and regulators/references
Parts:
- added JP11, JP2, JP3, JP4: JumpForCrystal, 4ms_SolderJumper:JUMPER_SMD_1x2_tiny_shorted, symbol 4ms_Net-tie:JumpForCrystal
- gave numbers to parts that had none: 6
Connections:
- net +12V: now also JP11.1 (A), JP2.1 (A), JP3.1 (A), JP4.1 (A); no longer C49.1, C55.1, C67.1, C81.1, R66.1, U13.3 (IN), U6.1 (VI), V1.3 (VI), V2.1 (VI)
- new net: C49.1, JP4.2 (B), V1.3 (VI)
- new net: C67.1, JP2.2 (B), R66.1, U13.3 (IN)
- new net: C81.1, JP3.2 (B), V2.1 (VI)
- new net: C55.1, JP11.2 (B), U6.1 (VI)
Other:
- note added: "TODO for v1.1rc2: [x] SD Card is rotated 180 degrees (compared to STS and kit Sampler) [x] Pot and CV ADC pins are not the same as kit version (swapped Length and Start Pos pots? swapped Bank and Sample CV??) - SWAP LENGTH AND START POTS. SWAP BANK AND SAMP [x] Left and Right outputs are swapped on kit version, so we should do the same here [x] Pressing REV shorts it out? [X] Add soft start to +/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"
- note removed: "TODO for v1.1rc2: [x] SD Card is rotated 180 degrees (compared to STS and kit Sampler) [x] Pot and CV ADC pins are not the same as kit version (swapped Length and Start Pos pots? swapped Bank and Sample CV??) - SWAP LENGTH AND START POTS. SWAP BANK AND SAMP [x] Left and Right outputs are swapped on kit version, so we should do the same here [x] Pressing REV shorts it out? [ ] Find out from Dan wh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"
- moved on the sheet: C49, C51, NT1, V1
