File: v1.1-rc-4_12HP/Sampler-built.kicad_sch (KiCad schematic)
At the start: 248 parts, among them J10 Eurorack_Power_10pin_Unshroud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, J11 3.5mm_Mono_Switched, J12 3.5mm_Mono_Switched, J13 3.5mm_Mono_Switched, J14 3.5mm_Mono_Switched, J15 3.5mm_Mono_Switched, J16 3.5mm_Mono_Switched, J17 3.5mm_Mono_Switched, J2 3.5mm_Mono_Switched, J3 Conn_01x04, J4 Conn_02x04, J6 3.5mm_Mono_Switched, J7 3.5mm_Mono_Switched, J8 3.5mm_Mono_Switched, J9 3.5mm_Mono_Switched, Q11 Si2347, Q12 Si2318, U1 TL072H, U10 TL072H, U11 TL072H, U12 TL072H, U13 AP62200WU-7, U14 TL072H, U15 TL072H, U16 TL072H, U18 STS SD card w/adaptor, U2 STM32F746IE, U3 TL072H, U4 SDRAM_IS42S16400J-6BLI-TR, U5 TL072H, U6 NCP51460SN33, U8 TL072H, U9 PCM3060PW, Y1 16MHz_18pF_FA238

Commit message: Updated todo list
Other:
- note added: "TODO for v1.1rc4: [X] Swap Left and Right output jacks (done on the PCB side) [ ] Wait for Dan's response if the pots need to have each their own single op amp There is a note in the pot section about this but it may be left over from earlier protos"
- note removed: "TODO for v1.1rc4: [X] Swap Left and Right output jacks (done on the PCB side)"
Changed lines of the file:
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@@
 		)
 	)
-	(text "TODO for v1.1rc4:\n[X] Swap Left and Right output jacks (done on the PCB side)"
+	(text "TODO for v1.1rc4:\n[X] Swap Left and Right output jacks (done on the PCB side)\n[ ] Wait for Dan's response if the pots need to have each their own single op amp\n	There is a note in the pot section about this but it may be left over from earlier\n	protos"
 		(exclude_from_sim no)
 		(at 377.698 797.052 0)

Commit message: Updated TODO list
Other:
- note added: "TODO for v1.1rc4: [X] Swap Left and Right output jacks (done on the PCB side)"
- note removed: "TODO for v1.1rc4: [X] Swap Left and Right output jacks (done on the PCB side) [ ] Wait for Dan's response if the pots need to have each their own single op amp There is a note in the pot section about this but it may be left over from earlier protos"
- note removed: "TODO: Use single op-amps for pots"
Changed lines of the file:
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@@
-		)
-	)
-	(text "TODO: Use single op-amps for pots"
-		(exclude_from_sim no)
-		(at 953.77 41.91 0)
-		(effects
-			(font
-				(size 2 2)
-				(thickness 0.4)
-				(bold yes)
-			)
-			(justify left bottom)
 		)
 	)
@@
 		)
 	)
-	(text "TODO for v1.1rc4:\n[X] Swap Left and Right output jacks (done on the PCB side)\n[ ] Wait for Dan's response if the pots need to have each their own single op amp\n	There is a note in the pot section about this but it may be left over from earlier\n	protos"
+	(text "TODO for v1.1rc4:\n[X] Swap Left and Right output jacks (done on the PCB side)"
 		(exclude_from_sim no)
 		(at 377.698 797.052 0)
