File: v1.1-rc-5_12HP/Sampler-built.kicad_sch (KiCad schematic)
At the start: 248 parts, among them J10 Eurorack_Power_10pin_Unshroud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, J11 3.5mm_Mono_Switched, J12 3.5mm_Mono_Switched, J13 3.5mm_Mono_Switched, J14 3.5mm_Mono_Switched, J15 3.5mm_Mono_Switched, J16 3.5mm_Mono_Switched, J17 3.5mm_Mono_Switched, J2 3.5mm_Mono_Switched, J3 Conn_01x04, J4 Conn_02x04, J6 3.5mm_Mono_Switched, J7 3.5mm_Mono_Switched, J8 3.5mm_Mono_Switched, J9 3.5mm_Mono_Switched, Q11 Si2347, Q12 Si2318, U1 TL072H, U10 TL072H, U11 TL072H, U12 TL072H, U13 AP62200WU-7, U14 TL072H, U15 TL072H, U16 TL072H, U18 STS SD card w/adaptor, U2 STM32F746IE, U3 TL072H, U4 SDRAM_IS42S16400J-6BLI-TR, U5 TL072H, U6 NCP51460SN33, U8 TL072H, U9 PCM3060PW, Y1 16MHz_18pF_FA238

Commit message: Removed old TODO informationfrom schematic
Other:
- note removed: "TODO for v1.1rc2: [x] SD Card is rotated 180 degrees (compared to STS and kit Sampler) [x] Pot and CV ADC pins are not the same as kit version (swapped Length and Start Pos pots? swapped Bank and Sample CV??) - SWAP LENGTH AND START POTS. SWAP BANK AND SAMP [x] Left and Right outputs are swapped on kit version, so we should do the same here [x] Pressing REV shorts it out? [X] Add soft start to +/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"
Changed lines of the file:
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@@
-		)
-	)
-	(text "TODO for v1.1rc2:\n[x] SD Card is rotated 180 degrees (compared to STS and kit Sampler)\n[x] Pot and CV ADC pins are not the same as kit version (swapped Length and Start Pos pots?\nswapped Bank and Sample CV??) - SWAP LENGTH AND START POTS. SWAP BANK AND SAMP\n[x] Left and Right outputs are swapped on kit version, so we should do the same here\n[x] Pressing REV shorts it out?\n[X] Add soft start to +/-12V\n[X] Add solder jumpers between +12v and all regulators/references"
-		(exclude_from_sim no)
-		(at 377.698 797.052 0)
-		(effects
-			(font
-				(size 10 10)
-				(thickness 2)
-				(bold yes)
-				(italic yes)
-			)
-			(justify left bottom)
 		)
 	)

Commit message: Updated majority of 0603 parts to be 0402 and matched library links so parts showup on the same line of the BOM
Parts:
- C1, C10, C11, C12, C13, C14, C15, C17, C18, C27, C28, C29, C3, C30, C31, C32, C33, C36, C41, C50, C53, C6, C7, C9: value 100nF_0402_16V -> 100nF_0402_50V; symbol 4ms_Capacitor:100nF_0402_16V -> 4ms_Capacitor:100nF_0402_50V
- C16, C20: value 100nF_0603_16V -> 100nF_0402_50V; footprint 4ms_Capacitor:C_0603 -> 4ms_Capacitor:C_0402; symbol 4ms_Capacitor:100nF_0603_16V -> 4ms_Capacitor:100nF_0402_50V; JLCPCB ID C14663 -> C1525; Manufacturer AVX Corporation -> Murata; Manufacturer 2 (none) -> Yageo; Part Number 0603YC104KAT2A -> GCM155R71C104KA55D; Part Number 2 (none) -> CC0402KRX7R7BB104
- C25, C26, C39, C42, C45, C47, C54, C58, C65, C66, C79, C83: value 0.1uF_0603_16V -> 100nF_0402_50V; footprint 4ms_Capacitor:C_0603 -> 4ms_Capacitor:C_0402; symbol 4ms_Capacitor:0.1uF_0603_16V -> 4ms_Capacitor:100nF_0402_50V; JLCPCB ID C14663 -> C1525; Manufacturer AVX Corporation -> Murata; Manufacturer 2 (none) -> Yageo; Part Number 0603YC104KAT2A -> GCM155R71C104KA55D; Part Number 2 (none) -> CC0402KRX7R7BB104
- C46: value 1nF_0603_50V -> 1nF_0402_50V; footprint 4ms_Capacitor:C_0603 -> 4ms_Capacitor:C_0402; symbol 4ms_Capacitor:1nF_0603_50V -> 4ms_Capacitor:1nF_0402_50V; JLCPCB ID C163508 -> C167632; Manufacturer Murata -> AVX Corportation; Part Number GRM1885C1H102JA01D -> 04025C102KAT2A; Specifications 1nF, 50V, 10%, C0G (NP0) or similar -> 1nF, 50V, 10%, X7R or similar
- C48, C57: value 220pF_0603_25V -> 220pF_0402_50V; footprint 4ms_Capacitor:C_0603 -> 4ms_Capacitor:C_0402; symbol 4ms_Capacitor:220pF_0603_25V -> 4ms_Capacitor:220pF_0402_50V; JLCPCB ID C1603 -> C327000; Part Number CC0603JRNPO9BN221 -> AC0402JPNPO9BN221; Specifications 220pF, Min 25V, C0G/NP0, 5% 0603 -> 220pF, 50V, 5%, X7R or X5R or similar
- C84: value 100pF_0603_50V -> 100pF_0402_50V; footprint 4ms_Capacitor:C_0603 -> 4ms_Capacitor:C_0402; symbol 4ms_Capacitor:100pF_0603_50V -> 4ms_Capacitor:100pF_0402_50V; JLCPCB ID C14858 -> C106200; Part Number CC0603JRNPO9BN101 -> CC0402JRNPO9BN101; Specifications 100pF, Min. 50V 10% NP0 or C0G -> 100pF, Min. 50V 5% NP0 or C0G
- R13, R3, R35, R5, R64, R68: value 2k_0603 -> 2k_0402; footprint 4ms_Resistor:R_0603 -> 4ms_Resistor:R_0402; symbol 4ms_Resistor_0603:2k_0603 -> 4ms_Resistor_0402:2k_0402; JLCPCB ID C105576 -> C60488; Part Number RC0603FR-072KL -> RC0402FR-072KL; Specifications 2k, 1%, 1/10W, 0603 -> 2k, 1%, 1/16W, 0402
- R15, R16, R17, R20, R58, R59, R62: value 47k_0603 -> 47k_0402; footprint 4ms_Resistor:R_0603 -> 4ms_Resistor:R_0402; symbol 4ms_Resistor_0603:47k_0603 -> 4ms_Resistor_0402:47k_0402; JLCPCB ID C105579 -> C93943; Part Number RC0603FR-0747KL -> RC0402FR-0747KL; Specifications 47k, 1%, 1/10W, 0603 -> 47k, 1%, 1/16W, 0402
- R21, R24, R25, R26, R32: value 100k_0603 -> 100k_0402; footprint 4ms_Resistor:R_0603 -> 4ms_Resistor:R_0402; symbol 4ms_Resistor_0603:100k_0603 -> 4ms_Resistor_0402:100k_0402; JLCPCB ID C14675 -> C60491; Part Number RC0603FR-07100KL -> RC0402FR-07100KL; Specifications 100k, 1%, 1/10W, 0603 -> 100k, 1%, 1/16W, 0402
- R29: value 20k_0603 -> 20k_0402; footprint 4ms_Resistor:R_0603 -> 4ms_Resistor:R_0402; symbol 4ms_Resistor_0603:20k_0603 -> 4ms_Resistor_0402:20k_0402; JLCPCB ID C105575 -> C93942; Part Number RC0603FR-0720KL -> RC0402FR-0720KL; Specifications 20k, 1%, 1/10W, 0603 -> 20k, 1%, 1/16W, 0402
- R31, R37: value 1M_0603 -> 1M_0402; footprint 4ms_Resistor:R_0603 -> 4ms_Resistor:R_0402; symbol 4ms_Resistor_0603:1M_0603 -> 4ms_Resistor_0402:1M_0402; JLCPCB ID C105578 -> C138033; Part Number RC0603FR-071ML -> RC0402FR-071ML; Specifications 1M, 1%, 1/10W, 0603 -> 1M, 1%, 1/16W, 0402
- R36, R60, R73, R74: value 10k_0603 -> 10k_0402; footprint 4ms_Resistor:R_0603 -> 4ms_Resistor:R_0402; symbol 4ms_Resistor_0603:10k_0603 -> 4ms_Resistor_0402:10k_0402; JLCPCB ID C98220 -> C60490; Part Number RC0603FR-0710KL -> RC0402FR-0710KL; Specifications 10k, 1%, 1/10W, 0603 -> 10k, 1%, 1/16W, 0402
- R56, R57, R61, R77, R78, R79, R80: value 33k_0603 -> 33k_0402; footprint 4ms_Resistor:R_0603 -> 4ms_Resistor:R_0402; symbol 4ms_Resistor_0603:33k_0603 -> 4ms_Resistor_0402:33k_0402; JLCPCB ID C126359 -> C138003; Part Number RC0603FR-0733KL -> RC0402FR-0733KL; Specifications 33k, 1%, 1/10W, 0603 -> 33k, 1%, 1/16W, 0402
- R63, R9: value 1k_0603 -> 1k_0402; footprint 4ms_Resistor:R_0603 -> 4ms_Resistor:R_0402; symbol 4ms_Resistor_0603:1k_0603 -> 4ms_Resistor_0402:1k_0402; JLCPCB ID C22548 -> C106235; Part Number RC0603FR-071KL -> RC0402FR-071KL; Specifications 1k, 1%, 1/10W, 0603 -> 1k, 1%, 1/16W, 0402
- R70, R71, R75: value 330Ω_0603 -> 330Ω_0402; footprint 4ms_Resistor:R_0603 -> 4ms_Resistor:R_0402; symbol 4ms_Resistor_0603:330Ω_0603 -> 4ms_Resistor_0402:330Ω_0402; JLCPCB ID C105881 -> C105875; Part Number RC0603FR-07330RL -> RC0402FR-07330RL; Specifications 330Ω, 1%, 1/10W, 0603 -> 330Ω, 1%, 1/16W, 0402

Commit message: Changed 16v 100nf caps to be 50v and apear on same BOM line
Parts:
- C1, C10, C11, C12, C13, C14, C15, C16, C17, C18, C20, C25, C26, C27, C28, C29, C3, C30, C31, C32, C33, C36, C39, C41, C42, C45, C47, C50, C53, C54, C58, C6, C65, C66, C7, C79, C83, C9: Alt JLCPCB ID (none) -> C77020; JLCPCB ID C1525 -> C307331; Manufacturer 2 Yageo -> (none); Part Number GCM155R71C104KA55D -> GRM155R71H104KE14D; Part Number 2 CC0402KRX7R7BB104 -> (none); Specifications 0.1uF, Min. 16V 10%, X7R or X5R or similar -> 0.1uF, Min. 50V 10%, X7R or X5R or similar

Commit message: Generated production files and submitted project
Parts:
- JP11, JP2, JP3, JP4: footprint 4ms_SolderJumper:JUMPER_SMD_1x2_tiny_shorted -> 4ms_SolderJumper:Net_Tie_0.16mm_6mil
